File: pcb/esp32-comp-tester.kicad_sch (KiCad schematic)
At the start: 20 parts, among them J1 PWR JST, J2 USB_A, J3 UART_JST, J4 ZIF Test Point Socket, SW1 SW_Push, SW2 SW_Push, U1 ESP32-WROOM-32, U2 AMS1117-3.3, U2 CH340G

Commit message: Updated Schematic
Parts:
- added C4: 0.1uF, symbol pspice:C
- added D1: LED, symbol Device:LED
- added J5: Screen SPI Data, symbol Connector:Conn_01x04_Pin
- added J6: Screen Power Pins, symbol Connector:Conn_01x03_Pin
- added J7: AVR-JTAG-10, Connector_IDC:IDC-Header_2x05_P2.54mm_Vertical, symbol Connector:AVR-JTAG-10
- added R7: 680, symbol Device:R
- added R8: 10k, symbol Device:R
- added SW3: Measure Push Button, symbol Switch:SW_Push
- added TP1: TP_A, TestPoint:TestPoint_Pad_D2.0mm, symbol Connector:TestPoint
- added TP2: TP_B, TestPoint:TestPoint_Pad_D2.0mm, symbol Connector:TestPoint
- added TP3: TP_C, TestPoint:TestPoint_Pad_D2.0mm, symbol Connector:TestPoint
- added TP4: TP_RX, TestPoint:TestPoint_Pad_D2.0mm, symbol Connector:TestPoint
- added TP5: TP_TX, TestPoint:TestPoint_Pad_D2.0mm, symbol Connector:TestPoint
- added TP6, TP7: TP_GND, TestPoint:TestPoint_Pad_D2.0mm, symbol Connector:TestPoint
- added TP8, TP9: TP_3.3V, TestPoint:TestPoint_Pad_D2.0mm, symbol Connector:TestPoint
- C3: value C -> 22uF
- C5, C6: value C -> 0.1uF
Connections:
- net +3.3V: now also D1.2 (A), J6.2 (Pin_2), J7.4 (VREF), J7.7 (VCC), R8.1, TP8.1, TP9.1
- net +5V: now also J6.3 (Pin_3)
- net ADC1_CH3_TP1: now also J4.8 (Pin_8), TP1.1; no longer J4.10 (Pin_10)
- net ADC1_CH6_TP2: now also J4.9 (Pin_9), TP2.1; no longer J4.8 (Pin_8)
- net ADC1_CH7_TP3: now also J4.10 (Pin_10), J7.9 (TDI), TP3.1; no longer J4.9 (Pin_9)
- net EN: now also C4.1, R8.2
- net ESP_RX: now also TP4.1
- net ESP_TX: now also TP5.1
- net GND: now also C4.2, J6.1 (Pin_1), J7.10 (GND), J7.2 (GND), R7.2, SW3.2, TP6.1, TP7.1
- net R1_TP3: now also J7.1 (TCK)
- net R2_TP2: now also J7.5 (TMS)
- net R2_TP3: now also J7.3 (TDO)
- net VSPI_CLK: now also J5.4 (Pin_4)
- net VSPI_CS: now also J5.1 (Pin_1)
- net VSPI_MISO: now also J5.3 (Pin_3)
- net VSPI_MOSI: now also J5.2 (Pin_2)
- net MEAS_PIN: now reaches U1.28 (IO17)
- net MEAS_PIN: now also SW3.1
- new net: D1.1 (K), R7.1
Other:
- note added: "JTAG Debugging Connector"
- note added: "Measure Physical Button"
- note added: "Power Section"
- note added: "Power Test Point Pads"
- note added: "Screen Connectors"

Commit message: Added V1 PCB
Parts:
- added TP10: GPIO_22, TestPoint:TestPoint_Pad_D2.0mm, symbol Connector:TestPoint
- added TP11: GPIO_21, TestPoint:TestPoint_Pad_D2.0mm, symbol Connector:TestPoint
- added TP12: GPIO_16, TestPoint:TestPoint_Pad_D2.0mm, symbol Connector:TestPoint
- added TP13, TP14: TP_3.3V, TestPoint:TestPoint_Pad_D2.0mm, symbol Connector:TestPoint
- added TP15: GPIO_36, TestPoint:TestPoint_Pad_D2.0mm, symbol Connector:TestPoint
- added TP16: SRST, TestPoint:TestPoint_Pad_D2.0mm, symbol Connector:TestPoint
- added TP17: TRST, TestPoint:TestPoint_Pad_D2.0mm, symbol Connector:TestPoint
- added TP18: CTS, TestPoint:TestPoint_Pad_D2.0mm, symbol Connector:TestPoint
- added TP19: DSR, TestPoint:TestPoint_Pad_D2.0mm, symbol Connector:TestPoint
- added TP20: RI, TestPoint:TestPoint_Pad_D2.0mm, symbol Connector:TestPoint
- added TP21: DCD, TestPoint:TestPoint_Pad_D2.0mm, symbol Connector:TestPoint
- added TP22: DTR, TestPoint:TestPoint_Pad_D2.0mm, symbol Connector:TestPoint
- added TP23: RTS, TestPoint:TestPoint_Pad_D2.0mm, symbol Connector:TestPoint
- added TP24: XI, TestPoint:TestPoint_Pad_D2.0mm, symbol Connector:TestPoint
- added TP25: X0, TestPoint:TestPoint_Pad_D2.0mm, symbol Connector:TestPoint
- added TP26: R232, TestPoint:TestPoint_Pad_D2.0mm, symbol Connector:TestPoint
- added TP27: V3_CH340g, TestPoint:TestPoint_Pad_D2.0mm, symbol Connector:TestPoint
- added TP28: SCS, TestPoint:TestPoint_Pad_D2.0mm, symbol Connector:TestPoint
- added TP29: SCK, TestPoint:TestPoint_Pad_D2.0mm, symbol Connector:TestPoint
- added TP30: SWP, TestPoint:TestPoint_Pad_D2.0mm, symbol Connector:TestPoint
- added TP31: SHD, TestPoint:TestPoint_Pad_D2.0mm, symbol Connector:TestPoint
- added TP32: SDI, TestPoint:TestPoint_Pad_D2.0mm, symbol Connector:TestPoint
- added TP33: SDO, TestPoint:TestPoint_Pad_D2.0mm, symbol Connector:TestPoint
- C1, C2, C3: footprint (none) -> Capacitor_SMD:C_1206_3216Metric
- C4, C5, C6: footprint (none) -> Capacitor_SMD:C_0603_1608Metric
- D1: footprint (none) -> LED_SMD:LED_1206_3216Metric
- J1, J3: footprint (none) -> Connector_PinSocket_2.54mm:PinSocket_1x02_P2.54mm_Vertical
- J2: footprint (none) -> Connector_USB:USB_A_Molex_48037-2200_Horizontal
- J4: footprint (none) -> Package_DIP:DIP-14_W7.62mm_Socket
- J5: footprint (none) -> Connector_JST:JST_EH_B4B-EH-A_1x04_P2.50mm_Vertical
- J6: footprint (none) -> Connector_JST:JST_EH_B3B-EH-A_1x03_P2.50mm_Vertical
- R1, R2, R3, R4, R5, R6, R7, R8: footprint (none) -> Resistor_SMD:R_1206_3216Metric
- SW1, SW2: footprint (none) -> Button_Switch_SMD:SW_SPST_B3S-1000
- SW3: footprint (none) -> Button_Switch_SMD:SW_SPST_B3S-1100
- renumbered U2 to U3
Connections:
- net ADC1_CH3_TP1: now also J4.10 (Pin_10), J4.9 (Pin_9); no longer J4.12 (Pin_12), J4.13 (Pin_13)
- net ADC1_CH6_TP2: now also J4.13 (Pin_13); no longer J4.9 (Pin_9)
- net ADC1_CH7_TP3: now also J4.12 (Pin_12); no longer J4.10 (Pin_10)
- net at U1.17 (SHD/SD2): now also TP31.1
- net at U1.18 (SWP/SD3): now also TP30.1
- net at U1.19 (SCS/CMD): now also TP28.1
- net at U1.20 (SCK/CLK): now also TP29.1
- net at U1.21 (SDO/SD0): now also TP33.1
- net at U1.22 (SDI/SD1): now also TP32.1
- net at U1.24 (IO2): now also TP13.1
- net at U1.26 (IO4): now also TP14.1
- net at U1.27 (IO16): now also TP12.1
- net at U1.33 (IO21): now also TP11.1
- net at U1.36 (IO22): now also TP10.1
- net at U1.4 (SENSOR_VP): now also TP15.1
- net at J7.6 (~{SRST}): now also TP16.1
- net at J7.8 (~{TRST}): now also TP17.1
- net at U3.10 (~{DSR}): now also TP19.1
- net at U3.11 (~{RI}): now also TP20.1
- net at U3.12 (~{DCD}): now also TP21.1
- net at U3.13 (~{DTR}): now also TP22.1
- net at U3.14 (~{RTS}): now also TP23.1
- net at U3.15 (R232): now also TP26.1
- net at U3.4 (V3): now also TP27.1
- net at U3.7 (XI): now also TP24.1
- net at U3.8 (XO): now also TP25.1
- net at U3.9 (~{CTS}): now also TP18.1
Other:
- moved on the sheet: C4, R8

Commit message: Little PCB Changes
Parts:
- TP14: value TP_3.3V -> GPIO_4
Changed lines of the file:
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@@
       (effects (font (size 1.27 1.27)) (justify left))
     )
-    (property "Value" "TP_3.3V" (at 163.195 75.565 90)
+    (property "Value" "GPIO_4" (at 163.195 75.565 90)
       (effects (font (size 1.27 1.27)) (justify left))
     )
