File: pcb/esp32-comp-tester.kicad_pcb (KiCad board)
At the start: 2 copper layers, 100 x 100 mm, 68 parts, among them J1 PWR JST, J2 USB_A, J4 ZIF Test Point Socket, J5 Screen SPI Data, J6 Screen Power Pins, J7 AVR-JTAG-10, SW1 SW_Push, SW2 SW_Push, U1 ESP32-WROOM-32, U2 AMS1117-3.3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

Commit message: Added inductor measurement
Parts:
- removed the REF** at (157.5, 111.8)

Commit message: Added quality and dissipation factors
Parts:
- renumbered UART to J3, Measure to SW3
Connections:
- SW3 pad 3: GND -> (no net)
Changed lines of the file:
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@@
     (property "ki_keywords" "connector")
     (attr through_hole)
-    (fp_text reference "UART" (at 0 -2.77) (layer "F.SilkS")
+    (fp_text reference "J3" (at 0 -2.77) (layer "F.SilkS")
         (effects (font (size 1 1) (thickness 0.15)))
     )
@@
     (property "ki_keywords" "switch normally-open pushbutton push-button")
     (attr smd)
-    (fp_text reference "Measure" (at 0 -5.42) (layer "F.SilkS")
+    (fp_text reference "SW3" (at 0 -5.42) (layer "F.SilkS")
         (effects (font (size 1 1) (thickness 0.15)))
     )
@@
     (pad "2" smd rect (at 3.98 1.33) (size 1.55 1.3) (layers "F.Cu" "F.Paste" "F.Mask")
       (net 2 "GND") (pinfunction "2") (pintype "passive"))
-    (pad "3" smd rect (at 0 3.17) (size 1.3 1.7) (layers "F.Cu" "F.Paste" "F.Mask")
-      (net 2 "GND"))
+    (pad "3" smd rect (at 0 3.17) (size 1.3 1.7) (layers "F.Cu" "F.Paste" "F.Mask"))
     (model "${KICAD6_3DMODEL_DIR}/Button_Switch_SMD.3dshapes/SW_SPST_B3S-1100.wrl"
       (offset (xyz 0 0 0))
